File: Netflix and Chill LEDs/Netflix and Chill LEDs.kicad_sch (KiCad schematic)
At the start: 0 parts

Commit message: placement and routing done
Parts:
- added C1, C10, C11, C12, C13, C14, C15, C16, C17, C18, C19, C2, C20, C21, C22, C23, C24, C25, C26, C27, C28, C29, C3, C30, C31, C32, C33, C34, C35, C36, C37, C38, C39, C4, C40, C41, C42, C43, C44, C45, C46, C47, C48, C49, C5, C50, C51, C52, C53, C54, C55, C56, C57, C58, C59, C6, C60, C61, C7, C8, C9: 1uF, Capacitor_SMD:C_0603_1608Metric, symbol Device:C_Small
- added D1, D10, D11, D12, D13, D14, D15, D16, D17, D18, D19, D2, D20, D21, D22, D23, D24, D25, D26, D27, D28, D29, D3, D30, D31, D32, D33, D34, D35, D36, D37, D38, D39, D4, D40, D41, D42, D43, D44, D45, D46, D47, D48, D49, D5, D50, D51, D52, D53, D54, D55, D56, D57, D58, D59, D6, D60, D61, D7, D8, D9: WS2812B, LED_SMD:LED_WS2812B_PLCC4_5.0x5.0mm_P3.2mm, symbol LED:WS2812B
Connections:
- new net: D39.2 (DOUT), D40.4 (DIN)
- new net: D38.2 (DOUT), D39.4 (DIN)
- new net: D49.2 (DOUT), D50.4 (DIN)
- new net: D48.2 (DOUT), D49.4 (DIN)
- new net: D28.2 (DOUT), D29.4 (DIN)
- new net: D27.2 (DOUT), D28.4 (DIN)
- new net: D51.2 (DOUT), D52.4 (DIN)
- new net: D50.2 (DOUT), D51.4 (DIN)
- new net: D19.2 (DOUT), D20.4 (DIN)
- new net: D18.2 (DOUT), D19.4 (DIN)
- new net: D22.2 (DOUT), D23.4 (DIN)
- new net: D21.2 (DOUT), D22.4 (DIN)
- new net: D58.2 (DOUT), D59.4 (DIN)
- new net: D57.2 (DOUT), D58.4 (DIN)
- new net: D44.2 (DOUT), D45.4 (DIN)
- new net: D43.2 (DOUT), D44.4 (DIN)
- new net: D26.2 (DOUT), D27.4 (DIN)
- new net: D1.2 (DOUT), D2.4 (DIN)
- new net: D37.2 (DOUT), D38.4 (DIN)
- new net: D31.2 (DOUT), D32.4 (DIN)
- new net: D30.2 (DOUT), D31.4 (DIN)
- new net: D52.2 (DOUT), D53.4 (DIN)
- new net: D29.2 (DOUT), D30.4 (DIN)
- new net: D47.2 (DOUT), D48.4 (DIN)
- new net: D13.2 (DOUT), D14.4 (DIN)
- new net: D12.2 (DOUT), D13.4 (DIN)
- new net: D25.2 (DOUT), D26.4 (DIN)
- new net: D11.2 (DOUT), D12.4 (DIN)
- new net: D10.2 (DOUT), D11.4 (DIN)
- new net: D10.4 (DIN), D9.2 (DOUT)
- new net: D8.2 (DOUT), D9.4 (DIN)
- new net: D7.2 (DOUT), D8.4 (DIN)
- new net: D54.2 (DOUT), D55.4 (DIN)
- new net: D53.2 (DOUT), D54.4 (DIN)
- new net: D6.2 (DOUT), D7.4 (DIN)
- new net: D20.2 (DOUT), D21.4 (DIN)
- new net: D60.2 (DOUT), D61.4 (DIN)
- new net: D36.2 (DOUT), D37.4 (DIN)
- new net: D35.2 (DOUT), D36.4 (DIN)
- new net: D33.2 (DOUT), D34.4 (DIN)
- new net: D32.2 (DOUT), D33.4 (DIN)
- new net: D40.2 (DOUT), D41.4 (DIN)
- new net: D3.2 (DOUT), D4.4 (DIN)
- new net: D2.2 (DOUT), D3.4 (DIN)
- new net: D46.2 (DOUT), D47.4 (DIN)
- new net: D59.2 (DOUT), D60.4 (DIN)
- new net: D56.2 (DOUT), D57.4 (DIN)
- new net: D34.2 (DOUT), D35.4 (DIN)
- new net: D5.2 (DOUT), D6.4 (DIN)
- new net: D4.2 (DOUT), D5.4 (DIN)
- new net: D23.2 (DOUT), D24.4 (DIN)
- new net: D55.2 (DOUT), D56.4 (DIN)
- new net: D14.2 (DOUT), D15.4 (DIN)
- new net: D24.2 (DOUT), D25.4 (DIN)
- new net: D15.2 (DOUT), D16.4 (DIN)
- new net: D42.2 (DOUT), D43.4 (DIN)
- new net: D41.2 (DOUT), D42.4 (DIN)
- new net: D45.2 (DOUT), D46.4 (DIN)
- new net: D17.2 (DOUT), D18.4 (DIN)
- new net: D16.2 (DOUT), D17.4 (DIN)
- new net +5V: C1.2, C10.2, C11.2, C12.2, C13.2, C14.2, C15.2, C16.2, C17.2, C18.2, C19.2, C2.2, C20.2, C21.2, C22.2, C23.2, C24.2, C25.2, C26.2, C27.2, C28.2, C29.2, C3.2, C30.2, C31.2, C32.2, C33.2, C34.2, C35.2, C36.2, C37.2, C38.2, C39.2, C4.2, C40.2, C41.2, C42.2, C43.2, C44.2, C45.2, C46.2, C47.2, C48.2, C49.2, C5.2, C50.2, C51.2, C52.2, C53.2, C54.2, C55.2, C56.2, C57.2, C58.2, C59.2, C6.2, C60.2, C61.2, C7.2, C8.2, C9.2, D1.1 (VDD), D10.1 (VDD), D11.1 (VDD), D12.1 (VDD), D13.1 (VDD), D14.1 (VDD), D15.1 (VDD), D16.1 (VDD), D17.1 (VDD), D18.1 (VDD), D19.1 (VDD), D2.1 (VDD), D20.1 (VDD), D21.1 (VDD), D22.1 (VDD), D23.1 (VDD), D24.1 (VDD), D25.1 (VDD), D26.1 (VDD), D27.1 (VDD), D28.1 (VDD), D29.1 (VDD), D3.1 (VDD), D30.1 (VDD), D31.1 (VDD), D32.1 (VDD), D33.1 (VDD), D34.1 (VDD), D35.1 (VDD), D36.1 (VDD), D37.1 (VDD), D38.1 (VDD), D39.1 (VDD), D4.1 (VDD), D40.1 (VDD), D41.1 (VDD), D42.1 (VDD), D43.1 (VDD), D44.1 (VDD), D45.1 (VDD), D46.1 (VDD), D47.1 (VDD), D48.1 (VDD), D49.1 (VDD), D5.1 (VDD), D50.1 (VDD), D51.1 (VDD), D52.1 (VDD), D53.1 (VDD), D54.1 (VDD), D55.1 (VDD), D56.1 (VDD), D57.1 (VDD), D58.1 (VDD), D59.1 (VDD), D6.1 (VDD), D60.1 (VDD), D61.1 (VDD), D7.1 (VDD), D8.1 (VDD), D9.1 (VDD)
- new net GND: C1.1, C10.1, C11.1, C12.1, C13.1, C14.1, C15.1, C16.1, C17.1, C18.1, C19.1, C2.1, C20.1, C21.1, C22.1, C23.1, C24.1, C25.1, C26.1, C27.1, C28.1, C29.1, C3.1, C30.1, C31.1, C32.1, C33.1, C34.1, C35.1, C36.1, C37.1, C38.1, C39.1, C4.1, C40.1, C41.1, C42.1, C43.1, C44.1, C45.1, C46.1, C47.1, C48.1, C49.1, C5.1, C50.1, C51.1, C52.1, C53.1, C54.1, C55.1, C56.1, C57.1, C58.1, C59.1, C6.1, C60.1, C61.1, C7.1, C8.1, C9.1, D1.3 (VSS), D10.3 (VSS), D11.3 (VSS), D12.3 (VSS), D13.3 (VSS), D14.3 (VSS), D15.3 (VSS), D16.3 (VSS), D17.3 (VSS), D18.3 (VSS), D19.3 (VSS), D2.3 (VSS), D20.3 (VSS), D21.3 (VSS), D22.3 (VSS), D23.3 (VSS), D24.3 (VSS), D25.3 (VSS), D26.3 (VSS), D27.3 (VSS), D28.3 (VSS), D29.3 (VSS), D3.3 (VSS), D30.3 (VSS), D31.3 (VSS), D32.3 (VSS), D33.3 (VSS), D34.3 (VSS), D35.3 (VSS), D36.3 (VSS), D37.3 (VSS), D38.3 (VSS), D39.3 (VSS), D4.3 (VSS), D40.3 (VSS), D41.3 (VSS), D42.3 (VSS), D43.3 (VSS), D44.3 (VSS), D45.3 (VSS), D46.3 (VSS), D47.3 (VSS), D48.3 (VSS), D49.3 (VSS), D5.3 (VSS), D50.3 (VSS), D51.3 (VSS), D52.3 (VSS), D53.3 (VSS), D54.3 (VSS), D55.3 (VSS), D56.3 (VSS), D57.3 (VSS), D58.3 (VSS), D59.3 (VSS), D6.3 (VSS), D60.3 (VSS), D61.3 (VSS), D7.3 (VSS), D8.3 (VSS), D9.3 (VSS)

Commit message: layout done
Parts:
- added J2: CONN_02, Connector_PinHeader_2.54mm:PinHeader_1x02_P2.54mm_Vertical, symbol SparkFun-Connectors:CONN_02
- added U1: PixelBlazePico, _Breadstick_Footprints:PixelBlazePico, symbol _Breadstick_Library:PixelBlazePico
Connections:
- net +5V: now also J2.2, U1.4 (5V)
- net GND: now also J2.1, U1.1 (GND)
- net at D1.4 (DIN): now also U1.2 (DATA)
Changed lines of the file:
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@@
     (stroke (width 0) (type default) (color 0 0 0 0))
   )
+  (wire (pts (xy 280.67 30.48) (xy 287.02 30.48))
+    (stroke (width 0) (type default) (color 0 0 0 0))
+  )
   (wire (pts (xy 444.5 121.92) (xy 449.58 121.92))
     (stroke (width 0) (type default) (color 0 0 0 0))
@@
     (stroke (width 0) (type default) (color 0 0 0 0))
   )
+  (wire (pts (xy 224.79 29.21) (xy 224.79 35.56))
+    (stroke (width 0) (type default) (color 0 0 0 0))
+  )
   (wire (pts (xy 455.93 175.26) (xy 457.2 175.26))
     (stroke (width 0) (type default) (color 0 0 0 0))
@@
     (stroke (width 0) (type default) (color 0 0 0 0))
   )
+  (wire (pts (xy 215.9 21.59) (xy 224.79 21.59))
+    (stroke (width 0) (type default) (color 0 0 0 0))
+  )
   (wire (pts (xy 284.48 182.88) (xy 287.02 182.88))
     (stroke (width 0) (type default) (color 0 0 0 0))
@@
     (stroke (width 0) (type default) (color 0 0 0 0))
   )
+  (wire (pts (xy 209.55 24.13) (xy 209.55 36.83))
+    (stroke (width 0) (type default) (color 0 0 0 0))
+  )
   (wire (pts (xy 368.3 53.34) (xy 369.57 53.34))
     (stroke (width 0) (type default) (color 0 0 0 0))
@@
     (stroke (width 0) (type default) (color 0 0 0 0))
   )
+  (wire (pts (xy 246.38 58.42) (xy 246.38 60.96))
+    (stroke (width 0) (type default) (color 0 0 0 0))
+  )
   (wire (pts (xy 314.96 21.59) (xy 314.96 22.86))
     (stroke (width 0) (type default) (color 0 0 0 0))
@@
     (stroke (width 0) (type default) (color 0 0 0 0))
   )
+  (wire (pts (xy 224.79 24.13) (xy 209.55 24.13))
+    (stroke (width 0) (type default) (color 0 0 0 0))
+  )
   (wire (pts (xy 322.58 152.4) (xy 327.66 152.4))
     (stroke (width 0) (type default) (color 0 0 0 0))
@@
     (stroke (width 0) (type default) (color 0 0 0 0))
   )
+  (wire (pts (xy 241.3 58.42) (xy 246.38 58.42))
+    (stroke (width 0) (type default) (color 0 0 0 0))
+  )
   (wire (pts (xy 347.98 53.34) (xy 349.25 53.34))
     (stroke (width 0) (type default) (color 0 0 0 0))
@@
     (stroke (width 0) (type default) (color 0 0 0 0))
   )
+  (wire (pts (xy 217.17 35.56) (xy 224.79 35.56))
+    (stroke (width 0) (type default) (color 0 0 0 0))
+  )
   (wire (pts (xy 436.88 143.51) (xy 436.88 144.78))
     (stroke (width 0) (type default) (color 0 0 0 0))
@@
     (stroke (width 0) (type default) (color 0 0 0 0))
   )
+  (wire (pts (xy 241.3 55.88) (xy 246.38 55.88))
+    (stroke (width 0) (type default) (color 0 0 0 0))
+  )
   (wire (pts (xy 335.28 173.99) (xy 335.28 175.26))
     (stroke (width 0) (type default) (color 0 0 0 0))
@@
     (stroke (width 0) (type default) (color 0 0 0 0))
   )
+  (wire (pts (xy 246.38 55.88) (xy 246.38 53.34))
+    (stroke (width 0) (type default) (color 0 0 0 0))
+  )
   (wire (pts (xy 429.26 144.78) (xy 430.53 144.78))
     (stroke (width 0) (type default) (color 0 0 0 0))
@@
     (stroke (width 0) (type default) (color 0 0 0 0))
   )
+  (wire (pts (xy 280.67 36.83) (xy 280.67 30.48))
+    (stroke (width 0) (type default) (color 0 0 0 0))
+  )
   (wire (pts (xy 476.25 114.3) (xy 477.52 114.3))
     (stroke (width 0) (type default) (color 0 0 0 0))
@@
     (stroke (width 0) (type default) (color 0 0 0 0))
   )
+  (wire (pts (xy 209.55 36.83) (xy 280.67 36.83))
+    (stroke (width 0) (type default) (color 0 0 0 0))
+  )
   (wire (pts (xy 394.97 175.26) (xy 396.24 175.26))
     (stroke (width 0) (type default) (color 0 0 0 0))
@@
     (pin "2")
   )
+  (symbol (lib_id "power:GND") (at 215.9 21.59 0) (mirror y) (unit 1)
+    (in_bom yes) (on_board yes)
+    (property "Reference" "#PWR0184" (id 0) (at 215.9 27.94 0)
+      (effects (font (size 1.27 1.27)) hide)
+    )
+    (property "Value" "GND" (id 1) (at 215.9 25.4 0))
+    (property "Footprint" "" (id 2) (at 215.9 21.59 0)
+      (effects (font (size 1.27 1.27)) hide)
+    )
+    (property "Datasheet" "" (id 3) (at 215.9 21.59 0)
+      (effects (font (size 1.27 1.27)) hide)
+    )
+    (pin "1")
+  )
   (symbol (lib_id "power:+5V") (at 436.88 52.07 0) (unit 1)
     (in_bom yes) (on_board yes)
@@
     (pin "1")
   )
+  (symbol (lib_id "SparkFun-Connectors:CONN_02") (at 238.76 58.42 0) (unit 1)
+    (in_bom yes) (on_board yes) (fields_autoplaced)
+    (property "Reference" "J2" (id 0) (at 236.22 46.99 0)
+      (effects (font (size 1.143 1.143)))
+    )
+    (property "Value" "CONN_02" (id 1) (at 236.22 49.53 0)
+      (effects (font (size 1.143 1.143)))
+    )
+    (property "Footprint" "Connector_PinHeader_2.54mm:PinHeader_1x02_P2.54mm_Vertical" (id 2) (at 238.76 52.07 0)
+      (effects (font (size 0.508 0.508)) hide)
+    )
+    (property "Datasheet" "" (id 3) (at 238.76 58.42 0)
+      (effects (font (size 1.27 1.27)) hide)
+    )
+    (property "Field4" "XXX-00000" (id 4) (at 236.22 53.34 0)
+      (effects (font (size 1.524 1.524)))
+    )
+    (pin "1")
+    (pin "2")
+  )
   (symbol (lib_id "Device:C_Small") (at 311.15 114.3 90) (unit 1)
     (in_bom yes) (on_board yes)
@@
     (pin "1")
   )
+  (symbol (lib_id "power:+5V") (at 246.38 53.34 0) (unit 1)
+    (in_bom yes) (on_board yes)
+    (property "Reference" "#PWR0186" (id 0) (at 246.38 57.15 0)
+      (effects (font (size 1.27 1.27)) hide)
+    )
+    (property "Value" "+5V" (id 1) (at 246.38 49.53 0))
+    (property "Footprint" "" (id 2) (at 246.38 53.34 0)
+      (effects (font (size 1.27 1.27)) hide)
+    )
+    (property "Datasheet" "" (id 3) (at 246.38 53.34 0)
+      (effects (font (size 1.27 1.27)) hide)
+    )
+    (pin "1")
+  )
   (symbol (lib_id "Device:C_Small") (at 351.79 83.82 90) (unit 1)
     (in_bom yes) (on_board yes)
@@
     (pin "1")
   )
+  (symbol (lib_id "_Breadstick_Library:PixelBlazePico") (at 245.11 25.4 0) (unit 1)
+    (in_bom yes) (on_board yes) (fields_autoplaced)
+    (property "Reference" "U1" (id 0) (at 245.745 15.24 0))
+    (property "Value" "PixelBlazePico" (id 1) (at 245.745 17.78 0))
+    (property "Footprint" "_Breadstick_Footprints:PixelBlazePico" (id 2) (at 224.79 21.59 0)
+      (effects (font (size 1.27 1.27)) hide)
+    )
+    (property "Datasheet" "" (id 3) (at 224.79 21.59 0)
+      (effects (font (size 1.27 1.27)) hide)
+    )
+    (pin "1")
+    (pin "2")
+    (pin "3")
+    (pin "4")
+  )
   (symbol (lib_id "power:GND") (at 375.92 68.58 0) (mirror y) (unit 1)
     (in_bom yes) (on_board yes)
@@
     (pin "1")
   )
+  (symbol (lib_id "power:+5V") (at 217.17 35.56 0) (unit 1)
+    (in_bom yes) (on_board yes)
+    (property "Reference" "#PWR0185" (id 0) (at 217.17 39.37 0)
+      (effects (font (size 1.27 1.27)) hide)
+    )
+    (property "Value" "+5V" (id 1) (at 217.17 31.75 0))
+    (property "Footprint" "" (id 2) (at 217.17 35.56 0)
+      (effects (font (size 1.27 1.27)) hide)
+    )
+    (property "Datasheet" "" (id 3) (at 217.17 35.56 0)
+      (effects (font (size 1.27 1.27)) hide)
+    )
+    (pin "1")
+  )
   (symbol (lib_id "power:GND") (at 469.9 175.26 0) (mirror y) (unit 1)
     (in_bom yes) (on_board yes)
@@
     (pin "1")
   )
+  (symbol (lib_id "power:GND") (at 246.38 60.96 0) (mirror y) (unit 1)
+    (in_bom yes) (on_board yes)
+    (property "Reference" "#PWR0187" (id 0) (at 246.38 67.31 0)
+      (effects (font (size 1.27 1.27)) hide)
+    )
+    (property "Value" "GND" (id 1) (at 246.38 64.77 0))
+    (property "Footprint" "" (id 2) (at 246.38 60.96 0)
+      (effects (font (size 1.27 1.27)) hide)
+    )
+    (property "Datasheet" "" (id 3) (at 246.38 60.96 0)
+      (effects (font (size 1.27 1.27)) hide)
+    )
+    (pin "1")
+  )
   (symbol (lib_id "power:GND") (at 335.28 38.1 0) (mirror y) (unit 1)
     (in_bom yes) (on_board yes)
@@
       (reference "#PWR0183") (unit 1) (value "GND") (footprint "")
     )
+    (path "/084f3856-23b2-4598-8566-68dc4c6d544e"
+      (reference "#PWR0184") (unit 1) (value "GND") (footprint "")
+    )
+    (path "/b1fa7bb1-a45b-4d26-96d4-baded4fe36a7"
+      (reference "#PWR0185") (unit 1) (value "+5V") (footprint "")
+    )
+    (path "/81b32070-8504-470f-a1b8-b624024dbe68"
+      (reference "#PWR0186") (unit 1) (value "+5V") (footprint "")
+    )
+    (path "/b721ccce-0f28-46c3-a505-ae46d3911be5"
+      (reference "#PWR0187") (unit 1) (value "GND") (footprint "")
+    )
     (path "/c32139d8-7c6b-4df8-9e4a-4044518a3357"
       (reference "C1") (unit 1) (value "1uF") (footprint "Capacitor_SMD:C_0603_1608Metric")
@@
       (reference "D61") (unit 1) (value "WS2812B") (footprint "LED_SMD:LED_WS2812B_PLCC4_5.0x5.0mm_P3.2mm")
     )
+    (path "/61a161a7-099c-45ec-bfdc-f7511b216678"
+      (reference "J2") (unit 1) (value "CONN_02") (footprint "Connector_PinHeader_2.54mm:PinHeader_1x02_P2.54mm_Vertical")
+    )
+    (path "/83d1b926-c112-43b9-b544-3c13bababd70"
+      (reference "U1") (unit 1) (value "PixelBlazePico") (footprint "_Breadstick_Footprints:PixelBlazePico")
+    )
   )
